File: backplane.sch (KiCad schematic (older format))
At the start: 6 parts, among them J1 Conn_01x02, J2 PCA

Commit message: heigharcal names should be correct accross all boards. layouts are together in the backplane.pcb file, except for the pi and PCA. ESC breakout layout tightened up.
Parts:
- removed J1: Conn_01x02, symbol Connector_Generic:Conn_01x02
- removed J2: PCA, symbol Connector_Generic:Conn_02x20_Counter_Clockwise
- added J?: PCA9685, symbol Connector_Generic:Conn_01x24
Connections:
- net labels added: +48V, +5P, GND, PWM0, PWM1, PWM2, PWM3, PWM4, PWM5
- net labels removed: SCL, SDA
- wire segments 15 -> 47
- no-connect marks 0 -> 1
