File: power_converter/buck.sch (KiCad schematic (older format))
At the start: 46 parts, among them J7 Conn_01x01, J8 Conn_01x01, Q1 Q_PMOS_GDS, U4 LTC2946CMS#PBF

Commit message: heigharcal names should be correct accross all boards. layouts are together in the backplane.pcb file, except for the pi and PCA. ESC breakout layout tightened up.
Parts:
- renumbered BC1 to BC?, BC2 to BC?, BC4 to BC?, BC3 to BC?, C13 to C?, C12 to C?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
